File: hardware/desk_timer.kicad_pcb (KiCad board)
At the start: 2 copper layers, 65 x 30.2 mm, 31 parts, among them J1 GT-USB-7010ASV, J2 Pin Headers,2x20,SMD,P2.54mm,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, J3 SWD, SW1 SW_Push, U1 STM32G0B1CBT6, U2 AMS1117-3.3, Y1 32.768 KHz, 10ppm, 12.5pf, Y2 8 MHz, 10ppm, 10pf

Commit message: Finished board
Parts:
- added 3V3: TestPoint_Pad_1.0x1.0mm, TestPoint:TestPoint_Pad_1.0x1.0mm, F.Cu at (133.5, 67.2)
- added BZ1: PKMCS0909E4000-R1, Buzzer_Beeper:Buzzer_Murata_PKMCS0909E, F.Cu at (93.2, 78.2)
- added D3: 1N4148WT, Diode_SMD:D_SOD-523, F.Cu at (103.2, 78.2)
- added Q1: 2SC4213, Package_TO_SOT_SMD:SOT-323_SC-70, F.Cu at (100.4, 76.6)
- added R7: 280R, Resistor_SMD:R_0402_1005Metric, F.Cu at (102.8, 74.8)
- J2: footprint Connector_PinHeader_2.54mm:PinHeader_2x20_P2.54mm_Vertical_SMD -> Connector_PinHeader_2.54mm:PinHeader_2x20_P2.54mm_Vertical
- J3: footprint Connector_PinHeader_2.54mm:PinHeader_2x04_P2.54mm_Horizontal -> Connector_PinHeader_2.54mm:PinHeader_1x04_P2.54mm_Horizontal
- moved J2 24.0 mm to (136.5, 90.2)
- moved R6 9.46 mm to (104.2, 69.8)
- moved SW1 3.22 mm to (82.0, 81.8)
- moved R3 3.22 mm to (85.7, 80.0)
- moved C10 3.22 mm to (85.6, 82.6)
- moved J3 2.82 mm to (90.2, 66.9)
- moved D1 1.58 mm to (133.5, 69.0)
- moved R4 1.12 mm to (133.5, 70.0)
Connections:
- net Net-(U1-PA0) renamed LED_STATUS
- J3 pad 1: +3V3 -> GND
- J3 pad 2: NRST -> SWCLK
- J3 pad 4: UART_TX -> +3V3
- U1 pad 30: unconnected-(U1-PC6-Pad30) -> PWM_OUT
Routing:
- net +5V: track 30.4 -> 75.0 mm, vias 2 -> 4
- net UART_TX: track 18.9 -> 0.00 mm, vias 1 -> 0
- net +3V3: track 112.9 -> 127.4 mm, vias 5 -> 6
- net UART_RX: track 13.7 -> 0.00 mm, vias 1 -> 0
- net Net-(BZ1--): track 0.00 -> 7.05 mm
- net GND: track 179.0 -> 185.2 mm, vias 11 -> 9
- net SWCLK: track 17.2 -> 23.0 mm, vias 1 -> 2
- net JOY_LEFT: track 12.4 -> 17.5 mm
- net SWDIO: track 14.8 -> 17.9 mm, vias 0 -> 1
- net PWM_OUT: track 0.00 -> 2.59 mm
- net Net-(Q1-B): track 0.00 -> 2.50 mm
- net OLED_SCK: track 9.38 -> 11.7 mm
- net JOY_UP: track 16.0 -> 18.4 mm
- net JOY_PRESS: track 14.6 -> 16.9 mm
- net OLED_MISO: track 10.0 -> 12.2 mm
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Other:
- board size 65 x 30.2 mm -> 65.1 x 30.3 mm
- board text added: "SWD"
- board text removed: "NRST"
- board text removed: "RX"
- board text removed: "TX"

Commit message: Reorganized repo
Parts:
- removed D3: 1N4148WT, Diode_SMD:D_SOD-523
- removed R6: 10k, Resistor_SMD:R_0402_1005Metric
- removed R7: 280R, Resistor_SMD:R_0402_1005Metric
- added R8: 300R, Resistor_SMD:R_1206_3216Metric_Pad1.30x1.75mm_HandSolder, F.Cu at (100.2, 75.2)
- added R9: 1K, Resistor_SMD:R_0402_1005Metric, F.Cu at (99.7, 81.0)
- J3: footprint Connector_PinHeader_2.54mm:PinHeader_1x04_P2.54mm_Horizontal -> Connector_PinHeader_2.54mm:PinHeader_1x07_P2.54mm_Horizontal
- moved C10 5.31 mm to (82.0, 86.5), turned to 0 degrees
- moved R3 5.29 mm to (85.0, 85.2)
- moved Q1 4.24 mm to (96.8, 78.8)
- moved BZ1 4.16 mm to (89.5, 76.4)
- moved J3 1.34 mm to (88.9, 66.6)
- moved J2 0.25 mm to (136.5, 90.0)
Connections:
- J3 pad 1: GND -> UART_RX
- J3 pad 2: SWCLK -> UART_TX
- J3 pad 3: SWDIO -> NRST
- J3 pad 4: +3V3 -> GND
Routing:
- net UART_RX: track 0.00 -> 19.8 mm, vias 0 -> 1
- net NRST: track 44.4 -> 61.2 mm
- net UART_TX: track 0.00 -> 16.6 mm, vias 0 -> 1
- net +3V3: track 127.4 -> 135.2 mm
- net +5V: track 75.0 -> 82.7 mm
- net SWCLK: track 23.0 -> 17.0 mm
- net GND: track 185.2 -> 180.9 mm
- net PWM_OUT: track 2.59 -> 5.13 mm
- net Net-(Q1-B): track 2.50 -> 4.47 mm
Other:
- board text added: "3V3"
- board text added: "NRST"
- board text added: "RX"
- board text added: "TX"
- board text added: "desk_timer rev_b dogfault"
- board text removed: "+3V3"
